File: LoRa_Sensor.kicad_sch (KiCad schematic)
At the start: 28 parts, among them IC1 BME688, J1 Conn_01x02_Pin, J2 TC2030-IDC-NL, U1 RAK3172_MODULE, U2 2462

Commit message: done for the day :)
Parts:
- C1, C2, C3, C8, C9: footprint Capacitor_SMD:C_0603_1608Metric -> Capacitor_SMD:C_0805_2012Metric
Changed lines of the file:
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@@
       (effects (font (size 1.27 1.27)) (justify right))
     )
-    (property "Footprint" "Capacitor_SMD:C_0603_1608Metric" (at 35.2552 142.24 0)
+    (property "Footprint" "Capacitor_SMD:C_0805_2012Metric" (at 35.2552 142.24 0)
       (effects (font (size 1.27 1.27)) hide)
     )
@@
       (effects (font (size 1.27 1.27)) (justify right))
     )
-    (property "Footprint" "Capacitor_SMD:C_0603_1608Metric" (at 22.5552 142.24 0)
+    (property "Footprint" "Capacitor_SMD:C_0805_2012Metric" (at 22.5552 142.24 0)
       (effects (font (size 1.27 1.27)) hide)
     )
@@
       (effects (font (size 1.27 1.27)) (justify left))
     )
-    (property "Footprint" "Capacitor_SMD:C_0603_1608Metric" (at 37.7952 46.99 0)
+    (property "Footprint" "Capacitor_SMD:C_0805_2012Metric" (at 37.7952 46.99 0)
       (effects (font (size 1.27 1.27)) hide)
     )
@@
       (effects (font (size 1.27 1.27)) (justify left))
     )
-    (property "Footprint" "Capacitor_SMD:C_0603_1608Metric" (at 139.3952 72.39 0)
+    (property "Footprint" "Capacitor_SMD:C_0805_2012Metric" (at 139.3952 72.39 0)
       (effects (font (size 1.27 1.27)) hide)
     )
@@
       (effects (font (size 1.27 1.27)) (justify left))
     )
-    (property "Footprint" "Capacitor_SMD:C_0603_1608Metric" (at 50.4952 46.99 0)
-      (effects (font (size 1.27 1.27)) hide)
-    )
+    (property "Footprint" "Capacitor_SMD:C_0805_2012Metric" (at 50.4952 46.99 0)
+      (effects (font (size 1.27 1.27)) hide)
+    )
